File: Yusynth4lfo1.kicad_pcb (KiCad board)
At the start: 2 copper layers, 91.9 x 110 mm, 72 parts, among them J1 Conn_01x13_Male, J2 Conn_01x13_Female, J3 Conn_02x05_Counter_Clockwise, J4 FM level, J5 270°, J6 180°, J7 0°, J8 90°, Q1 BC547C, Q2 BC557C, Q3 BC557C, Q4 BC547C, Q5 BC547C, Q6 BC547C, SW1 SW_Push_DPDT, U1 LM13700, U2 TL074, U3 TL074

Commit message: nouvelle version
Routing:
- net +12V: track 226.4 -> 225.5 mm

Commit message: derniere version vérifié
Parts:
- removed REF** (x2): MountingHole_3.2mm_M3, MountingHole:MountingHole_3.2mm_M3
- added G***: LOGO, Logos:Gaston-Music1, F.Cu at (28.7, 45.7)
- added H1: MountingHole, MountingHole:MountingHole_3.2mm_M3, F.Cu at (104.2, 43.7)
- added H2: MountingHole, MountingHole:MountingHole_3.2mm_M3, F.Cu at (156.1, 43.7)
- Q1, Q2, Q3, Q4, Q5, Q6: footprint Package_TO_SOT_THT:TO-92_Inline -> Package_TO_SOT_THT:TO-92_HandSolder
- moved R20 1.20 mm to (137.4, 59.2)
- moved R23 0.40 mm to (137.3, 54.7)
- moved RV1 0.07 mm to (88.0, 54.0)
- moved R29 0.06 mm to (107.8, 119.6)
- moved J4 0.06 mm to (93.0, 116.0)
Connections:
- J1 pad 6: output level2 CW -> output level1 WP
- J1 pad 8: output level1 WP -> output level2 CW
- J2 pad 7: Net-(RV1-Pad1) -> Net-(J2-Pad7)
- J2 pad 8: Net-(RV1-Pad4) -> Net-(RV1-Pad6)
- J2 pad 9: Net-(RV1-Pad5) -> Net-(J2-Pad9)
- J4 pad TN: (no net) -> unconnected-(J4-PadTN)
- J5 pad TN: (no net) -> unconnected-(J5-PadTN)
- J6 pad TN: (no net) -> unconnected-(J6-PadTN)
- J7 pad TN: (no net) -> unconnected-(J7-PadTN)
- J8 pad TN: (no net) -> unconnected-(J8-PadTN)
- RV1 pad 1: Net-(RV1-Pad1) -> GND
- RV1 pad 3: GND -> Net-(J2-Pad9)
- RV1 pad 4: Net-(RV1-Pad4) -> GND
- RV1 pad 5: Net-(RV1-Pad5) -> Net-(J2-Pad7)
- RV1 pad 6: GND -> Net-(RV1-Pad6)
- RV4 pad 1: Net-(J4-PadT) -> GND
- RV4 pad 3: GND -> Net-(J4-PadT)
Routing:
- net Net-(J2-Pad9): track 0.00 -> 27.5 mm
- net output level1 WP: track 25.9 -> 52.8 mm
- net Net-(RV1-Pad6): track 0.00 -> 21.1 mm
- net Net-(RV1-Pad5): track 20.8 -> 0.00 mm
- net Net-(RV1-Pad4): track 18.5 -> 0.00 mm
- net Net-(J2-Pad7): track 0.00 -> 17.6 mm
- net Net-(RV1-Pad1): track 16.1 -> 0.00 mm
- net Net-(R23-Pad1): track 35.5 -> 29.9 mm
- net Net-(J4-PadT): track 51.0 -> 45.6 mm
- net output level2 CW: track 70.9 -> 66.5 mm
- net +12V: track 225.5 -> 229.5 mm
- net 0°: track 26.7 -> 30.4 mm
- net Net-(Q6-Pad2): track 5.92 -> 7.19 mm
- net Net-(Q5-Pad2): track 14.8 -> 16.1 mm
- net Net-(Q4-Pad2): track 5.36 -> 4.09 mm
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Other:
- board size 91.9 x 110 mm -> 142.4 x 128.4 mm
- board text added: "0°"
- board text added: "180°"
- board text added: "270°"
- board text added: "90°"
- board text added: "CV FM"
- board text added: "FM LEVEL"
- board text added: "JLCJLCJLCJLC"
- board text added: "OUTPUT LEVEL"
- board text added: "QUADRATURE-LFO"
- board text added: "RATE"
- board text added: "Yusynth"
